File: pcb/scot-resolver.kicad_pcb (KiCad board)
At the start: 2 copper layers, 146 parts, among them IC1 AD8692ARMZ, IC10 AD2S1210, IC2 AD8397ARZ, IC3 AD8692ARMZ, IC4 TSR1, IC5 AD8692ARMZ, IC6 AD8692ARMZ, IC7 AD8692ARMZ, IC8 MCP2562, IC9 STM32F0xxKxTx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

Commit message: WIP.
Parts:
- moved R39 1.62 mm to (135.3, 104.2)
- moved C60 0.92 mm to (133.8, 90.9)
- moved C66 0.70 mm to (135.4, 105.2), turned to 180 degrees
Routing:
- net GND: track 187.5 -> 261.1 mm, vias 7 -> 12
- net /CAN TXRX/3.3V_MCU: track 139.9 -> 196.7 mm, vias 9 -> 12
- net /Resolver Exciter/AD2S1210_VREF: track 43.6 -> 89.9 mm, vias 10 -> 11
- net /Microcontroller & Interface/5V_RESOLVER_ANALOGUE: track 161.3 -> 200.6 mm, vias 11 -> 12
- net /Microcontroller & Interface/~DOT: track 38.4 -> 67.5 mm, vias 4 -> 6
- net /Microcontroller & Interface/5V_RESOLVER_DIGITAL: track 5.06 -> 30.8 mm, vias 0 -> 2
- net Net-(IC9-Pad4): track 1.75 -> 27.1 mm
- net /Microcontroller & Interface/UART_DEBUG_TX: track 5.83 -> 20.7 mm
- net /Microcontroller & Interface/UART_DEBUG_RX: track 6.29 -> 20.0 mm
- net GNDA: track 377.8 -> 385.6 mm
- net /Resolver Receiver COS+/AD2S1210_INPUT: track 32.5 -> 38.6 mm
- net /Microcontroller & Interface/INC_A: track 0.00 -> 5.46 mm
- net /Microcontroller & Interface/INC_B: track 0.00 -> 5.28 mm
- net /Microcontroller & Interface/INC_NM: track 0.00 -> 5.21 mm
- net Net-(C66-Pad1): track 0.00 -> 5.12 mm
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
Commit message: WIP (nearly there!)
Parts:
- added H1: MountingHole, agg:M3_MOUNT, F.Cu at (135.0, 57.4)
- added H2: MountingHole, agg:M3_MOUNT, F.Cu at (135.0, 127.4)
- moved P1 30.4 mm to (87.6, 124.6), turned to 90 degrees
- moved J7 11.7 mm to (87.6, 114.4), turned to 180 degrees
- moved D4 8.56 mm to (119.9, 116.5)
- moved R38 8.09 mm to (119.9, 111.9)
- moved D5 7.85 mm to (126.4, 116.5)
- moved D3 7.83 mm to (132.9, 116.5)
- moved R40 7.19 mm to (126.4, 111.9)
- moved R37 6.54 mm to (132.9, 111.9)
- moved D6 4.93 mm to (108.6, 120.4)
- moved D7 4.74 mm to (99.6, 120.4)
- moved J2 4.32 mm to (86.1, 98.8)
- moved R41 4.14 mm to (108.6, 115.7)
- moved J3 4.10 mm to (86.1, 86.6)
- moved R42 4.06 mm to (99.6, 115.7)
Routing:
- net /Microcontroller & Interface/SWD_IO: track 10.1 -> 45.7 mm
- net /Microcontroller & Interface/SWD_CLK: track 10.3 -> 43.5 mm
- net /CAN TXRX/3.3V_MCU: track 196.7 -> 225.5 mm
- net Net-(IC9-Pad4): track 27.1 -> 51.4 mm, vias 1 -> 2
- net GND: track 261.1 -> 278.8 mm, vias 12 -> 11
- net /Resolver Exciter/AD2S1210_VREF: track 89.9 -> 107.1 mm
- net /Microcontroller & Interface/INC_A: track 5.46 -> 18.6 mm
- net GNDA: track 385.6 -> 397.2 mm, vias 83 -> 82
- net /Microcontroller & Interface/INC_B: track 5.28 -> 13.4 mm
- net /Microcontroller & Interface/UART_DEBUG_RX: track 20.0 -> 27.0 mm
- net AVCC: track 84.1 -> 90.0 mm
- net /Microcontroller & Interface/INC_NM: track 5.21 -> 10.1 mm
- net /Microcontroller & Interface/~LOT: track 65.5 -> 61.0 mm
- net /CAN TXRX/CAN_L: track 23.7 -> 19.7 mm
- net /Microcontroller & Interface/UART_DEBUG_TX: track 20.7 -> 24.6 mm
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Other:
- board outline added: 108.5 x 79.2 mm
- board text added: "CAN"
- board text added: "DC"
- board text added: "Feb 2020"
- board text added: "Phil M0DNY"
- board text added: "SCOT Resolver I/F"
- board text removed: "CAN In"
- board text removed: "CAN Out"

Commit message: WIP.
Routing:
- net GNDA: track 397.2 -> 480.2 mm, vias 82 -> 79
- net /Resolver Exciter/AD2S1210_VREF: track 107.1 -> 178.8 mm, vias 11 -> 17
- net /Microcontroller & Interface/5V_RESOLVER_ANALOGUE: track 200.6 -> 201.6 mm
Other:
- board text added: "COS"
- board text added: "EXC"
- board text added: "G"
- board text added: "H"
- board text added: "L"
- board text added: "R"
- board text added: "SIN"
- board text added: "T"

Commit message: WIP..
Parts:
- added C69: 100n, Capacitor_SMD:C_0402_1005Metric, F.Cu at (92.6, 121.4)
- added G***: LOGO, scot_logo:scot_logo, F.Cu at (152.0, 95.1)
Routing:
- net GND: track 278.8 -> 283.3 mm
- net Net-(C69-Pad1): track 51.4 -> 53.3 mm
- net /Microcontroller & Interface/A1: track 39.7 -> 40.4 mm
- net /Resolver Exciter/AD2S1210_EXC-: track 25.1 -> 24.6 mm
- net GNDA: track 480.2 -> 480.6 mm, vias 79 -> 78
Other:
- board size 108.5 x 79.2 mm -> 108.6 x 79.4 mm
- rule trace_min: 0.2 -> 0.15
- rule via_min_size: 0.4 -> 0.3

Commit message: Sent to fab (fab5)
Parts:
- removed G***: LOGO, scot_logo:scot_logo
- moved U1 5.84 mm to (151.3, 65.9)
- moved C21 5.84 mm to (146.1, 64.2)
- moved C23 5.84 mm to (146.1, 67.6)
- moved R20 5.62 mm to (127.6, 62.3), turned to 270 degrees
- moved C26 3.66 mm to (180.4, 63.5)
- moved U2 3.66 mm to (177.0, 64.7)
- moved C20 3.66 mm to (174.4, 64.7)
- moved R18 3.66 mm to (180.1, 59.7)
- moved R19 3.66 mm to (176.7, 59.7)
- moved C24 3.66 mm to (176.0, 61.0)
- moved D6 3.05 mm to (108.6, 123.4)
- moved D7 3.05 mm to (99.6, 123.4)
- moved R41 3.05 mm to (108.6, 118.7)
- moved R42 3.05 mm to (99.6, 118.7)
- moved D2 2.07 mm to (126.1, 58.9), turned to 180 degrees
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Connections:
- D2 pad 1: GND -> Net-(D2-Pad1)
- D2 pad 2: Net-(D2-Pad2) -> +15V
- R20 pad 1: Net-(D2-Pad2) -> Net-(D2-Pad1)
- R20 pad 2: +15V -> GND
Routing:
- net GNDA: track 480.6 -> 462.5 mm
- net /Microcontroller & Interface/5V_RESOLVER_ANALOGUE: track 201.6 -> 193.4 mm
- net AVCC: track 90.0 -> 84.9 mm
- net /Power Supplies/12V_EXCITER: track 104.9 -> 101.4 mm
- net /Microcontroller & Interface/~LOT: track 60.9 -> 63.9 mm
- net /Microcontroller & Interface/~DOT: track 64.6 -> 67.7 mm
- net GND: track 283.3 -> 280.8 mm
- net Net-(D2-Pad1): track 0.00 -> 2.43 mm
- net Net-(D2-Pad2): track 2.16 -> 0.00 mm
- net /Microcontroller & Interface/INC_NM: track 10.1 -> 11.3 mm
- net /Microcontroller & Interface/INC_B: track 13.2 -> 14.5 mm
- net /Microcontroller & Interface/INC_A: track 18.9 -> 19.4 mm
- net /CAN TXRX/3.3V_MCU: track 225.5 -> 226.0 mm
Other:
- board text added: "15V"
- board text removed: "15V OK"
