File: pcb/scot-resolver-can-txrx.sch (KiCad schematic (older format))
At the start: 4 parts, among them IC8 MCP2562

Commit message: WIP PCB v2.
Parts:
- added C?: 4u7/5V, Capacitor_SMD:C_0805_2012Metric_Pad1.15x1.40mm_HandSolder, symbol Device:C
- added JP?: SolderJumper_2_Open, Jumper:SolderJumper-2_P1.3mm_Open_RoundedPad1.0x1.5mm, symbol Jumper:SolderJumper_2_Open
- C53: value 100n -> 100n/3V3; footprint Capacitor_SMD:C_0402_1005Metric -> Capacitor_SMD:C_0603_1608Metric_Pad1.05x0.95mm_HandSolder
- C54: value 100n -> 100n/5V; footprint Capacitor_SMD:C_0402_1005Metric -> Capacitor_SMD:C_0603_1608Metric_Pad1.05x0.95mm_HandSolder
- IC8: footprint agg:DFN-8-EP-MICROCHIP -> agg:SOIC-8
Connections:
- net 5V_CAN: now also C?.2
- net CAN_H: now also JP?.2 (B); no longer R36.1
- net GND: now also C?.1
- new net: JP?.1 (A), R36.1
Other:
- note removed: "Only fit 120R for bus termination."
- moved on the sheet: C53, C54
Changed lines of the file:
@@
 F 0 "IC8" H 5300 3185 50  0000 C CNN
 F 1 "MCP2562" H 5300 3276 50  0000 C CNN
-F 2 "agg:DFN-8-EP-MICROCHIP" H 5000 3200 50  0001 L CNN
+F 2 "agg:SOIC-8" H 5000 3200 50  0001 L CNN
 F 3 "http://ww1.microchip.com/downloads/en/DeviceDoc/20005167C.pdf" H 5000 3100 50  0001 L CNN
 F 4 "" H 5000 3000 50  0001 L CNN "Farnell"
@@
 L Device:C C?
 U 1 1 5E4915E0
-P 6200 4350
+P 5950 4350
 AR Path="/5E4915E0" Ref="C?"  Part="1"
 AR Path="/5E4877AC/5E4915E0" Ref="C53"  Part="1"
-F 0 "C53" H 6315 4396 50  0000 L CNN
-F 1 "100n" H 6315 4305 50  0000 L CNN
-F 2 "Capacitor_SMD:C_0402_1005Metric" H 6238 4200 50  0001 C CNN
-F 3 "~" H 6200 4350 50  0001 C CNN
-	1    6200 4350
+F 0 "C53" H 6065 4396 50  0000 L CNN
+F 1 "100n/3V3" H 6065 4305 50  0000 L CNN
+F 2 "Capacitor_SMD:C_0603_1608Metric_Pad1.05x0.95mm_HandSolder" H 5988 4200 50  0001 C CNN
+F 3 "~" H 5950 4350 50  0001 C CNN
+	1    5950 4350
 	1    0    0    -1
 $EndComp
@@
 L Device:C C?
 U 1 1 5E4915E6
-P 6550 3850
+P 6100 3850
 AR Path="/5E4915E6" Ref="C?"  Part="1"
 AR Path="/5E4877AC/5E4915E6" Ref="C54"  Part="1"
-F 0 "C54" H 6665 3896 50  0000 L CNN
-F 1 "100n" H 6665 3805 50  0000 L CNN
-F 2 "Capacitor_SMD:C_0402_1005Metric" H 6588 3700 50  0001 C CNN
-F 3 "~" H 6550 3850 50  0001 C CNN
-	1    6550 3850
+F 0 "C54" H 6215 3896 50  0000 L CNN
+F 1 "100n/5V" H 6215 3805 50  0000 L CNN
+F 2 "Capacitor_SMD:C_0603_1608Metric_Pad1.05x0.95mm_HandSolder" H 6138 3700 50  0001 C CNN
+F 3 "~" H 6100 3850 50  0001 C CNN
+	1    6100 3850
 	1    0    0    -1
 $EndComp
@@
 Text HLabel 3300 3550 0    50   Input ~ 0
 CAN_L
-Text HLabel 3300 3950 0    50   Input ~ 0
+Text HLabel 3300 4350 0    50   Input ~ 0
 CAN_H
 Wire Wire Line
@@
 	3800 3550 3800 3600
 Wire Wire Line
-	3300 3950 3800 3950
-Wire Wire Line
-	3800 3950 3800 3900
+	3300 4350 3800 4350
 Wire Wire Line
 	4300 3700 4300 3550
@@
 Connection ~ 3800 3550
 Wire Wire Line
-	3800 3950 4300 3950
-Wire Wire Line
-	4300 3950 4300 3800
+	3800 4350 4300 4350
 Wire Wire Line
 	4300 3800 4900 3800
-Connection ~ 3800 3950
-Text Notes 4650 4100 2    50   ~ 0
-Only fit 120R for bus termination.
+Connection ~ 3800 4350
 Text HLabel 6850 3050 2    50   Input ~ 0
 CAN_MCU_RXD
@@
 5V_CAN
 Wire Wire Line
-	6550 3700 6550 3600
+	6100 3700 6100 3600
 Wire Wire Line
-	5800 3600 6200 3600
+	5800 3600 5950 3600
 Wire Wire Line
-	6550 4100 6550 4000
+	6100 4100 6100 4000
 Wire Wire Line
-	6550 4100 6850 4100
+	6100 4100 6700 4100
 Wire Wire Line
-	6850 4600 6200 4600
+	6850 4600 5950 4600
 Wire Wire Line
-	6200 4600 6200 4500
+	5950 4600 5950 4500
 Wire Wire Line
-	6200 4200 6200 3600
-Connection ~ 6200 3600
+	5950 4200 5950 3600
+Connection ~ 5950 3600
 Wire Wire Line
-	6200 3600 6550 3600
+	5950 3600 6100 3600
 Wire Wire Line
-	5950 3700 5950 4100
+	5850 3700 5850 4100
 Wire Wire Line
-	5950 4100 6550 4100
+	5850 4100 6100 4100
 Wire Wire Line
-	5700 3700 5950 3700
-Connection ~ 6550 4100
+	5700 3700 5850 3700
+Connection ~ 6100 4100
 Wire Wire Line
 	5750 3800 5750 4600
 Wire Wire Line
-	5750 4600 6200 4600
-Connection ~ 6200 4600
+	5750 4600 5950 4600
+Connection ~ 5950 4600
 $Comp
 L power:GND #PWR0136
@@
 $EndComp
 Wire Wire Line
-	6550 3600 6850 3600
+	6100 3600 6700 3600
 Wire Wire Line
 	6850 3600 6850 3550
-Connection ~ 6550 3600
+Connection ~ 6100 3600
+$Comp
+L Device:C C?
+U 1 1 5ECCE60D
+P 6700 3850
+AR Path="/5ECCE60D" Ref="C?"  Part="1"
+AR Path="/5E4877AC/5ECCE60D" Ref="C?"  Part="1"
+F 0 "C?" H 6815 3896 50  0000 L CNN
+F 1 "4u7/5V" H 6815 3805 50  0000 L CNN
+F 2 "Capacitor_SMD:C_0805_2012Metric_Pad1.15x1.40mm_HandSolder" H 6738 3700 50  0001 C CNN
+F 3 "~" H 6700 3850 50  0001 C CNN
+	1    6700 3850
+	1    0    0    -1
+$EndComp
+Wire Wire Line
+	6700 3700 6700 3600
+Connection ~ 6700 3600
+Wire Wire Line
+	6700 3600 6850 3600
+Wire Wire Line
+	6700 4000 6700 4100
+Connection ~ 6700 4100
+Wire Wire Line
+	6700 4100 6850 4100
+$Comp
+L Jumper:SolderJumper_2_Open JP?
+U 1 1 5ECD2E93
+P 3800 4100
+F 0 "JP?" V 3754 4168 50  0000 L CNN
+F 1 "SolderJumper_2_Open" V 3845 4168 50  0000 L CNN
+F 2 "Jumper:SolderJumper-2_P1.3mm_Open_RoundedPad1.0x1.5mm" H 3800 4100 50  0001 C CNN
+F 3 "~" H 3800 4100 50  0001 C CNN
+	1    3800 4100
+	0    1    1    0
+$EndComp
+Wire Wire Line
+	3800 3900 3800 3950
+Wire Wire Line
+	3800 4250 3800 4350
+Wire Wire Line
+	4300 3800 4300 4350
 $EndSCHEMATC

Commit message: pcb: Add 10u to VREF, all 0402->0603
Parts:
- gave numbers to parts that had none: 2
Changed lines of the file:
@@
 P 6700 3850
 AR Path="/5ECCE60D" Ref="C?"  Part="1"
-AR Path="/5E4877AC/5ECCE60D" Ref="C?"  Part="1"
-F 0 "C?" H 6815 3896 50  0000 L CNN
+AR Path="/5E4877AC/5ECCE60D" Ref="C38"  Part="1"
+F 0 "C38" H 6815 3896 50  0000 L CNN
 F 1 "4u7/5V" H 6815 3805 50  0000 L CNN
 F 2 "Capacitor_SMD:C_0805_2012Metric_Pad1.15x1.40mm_HandSolder" H 6738 3700 50  0001 C CNN
@@
 	6700 4100 6850 4100
 $Comp
-L Jumper:SolderJumper_2_Open JP?
+L Jumper:SolderJumper_2_Open JP2
 U 1 1 5ECD2E93
 P 3800 4100
-F 0 "JP?" V 3754 4168 50  0000 L CNN
+F 0 "JP2" V 3754 4168 50  0000 L CNN
 F 1 "SolderJumper_2_Open" V 3845 4168 50  0000 L CNN
 F 2 "Jumper:SolderJumper-2_P1.3mm_Open_RoundedPad1.0x1.5mm" H 3800 4100 50  0001 C CNN
